Commit message: good

File: cartpole1l.urdf (robot description, URDF)
Before this commit: robot physics, 4 links, 3 joints
Links:
- removed link pole1
- link cart: mass 5.0 -> 1
- link pole: mass 1.0 -> 10
- link slideBar: geometry visual box size=30 0.05 0.05
Joints:
- removed joint pole_to_pole
- joint cart_to_pole: axis 0 1 0 -> 1 0 0; limit effort=1000.0 velocity=5 -> lower=-15 upper=15 effort=1000.0 velocity=5
- joint slider_to_cart: axis 1 0 0 -> 0 1 0; limit lower=-4 upper=4 effort=1000.0 velocity=100 -> lower=-15 upper=15 effort=1000.0 velocity=5

Commit message: move mass to the end -> easier

File: cartpole1l.urdf (robot description, URDF)
Before this commit: robot physics, 3 links, 2 joints
Links:
- link cart: mass 1 -> 10
- link pole: mass 10 -> 1.0
Joints:
- joint cart_to_pole: limit lower=-15 upper=15 effort=1000.0 velocity=5 -> lower=-1500 upper=1500 effort=1000.0 velocity=5000
- joint slider_to_cart: limit lower=-15 upper=15 effort=1000.0 velocity=5 -> lower=-1500 upper=1500 effort=1000.0 velocity=5000

File: cartpole2l.urdf (robot description, URDF)
Before this commit: robot physics, 4 links, 3 joints
Links:
- link cart: mass 5.0 -> 10.0
Joints:
- joint cart_to_pole: limit effort=1000.0 velocity=5 -> lower=-1500 upper=1500 effort=10000.0 velocity=5000
- joint pole_to_pole: limit effort=1000.0 velocity=5 -> lower=-1500 upper=1500 effort=10000.0 velocity=5000
- joint slider_to_cart: limit lower=-4 upper=4 effort=1000.0 velocity=100 -> lower=-1500 upper=1500 effort=10000.0 velocity=5000
